Commit message: Incorporado controlador ackermann e URDF adaptados para o modelo da bicicleta

File: Jetson/catkin_ws/src/robot_control/robot_description/urdf/Ackermann_robot.urdf (robot description, URDF)
Before this commit: robot Ackermann_robot, 10 links, 9 joints
Links:
- link chassi_link: geometry collision box size=0.22043 0.27703 0.12452; visual mesh filename=package://robot_control/robot_description/meshes/stl/Base.s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 scale=1.0 1.0 1.0
- link link_acker_front_left: geometry visual mesh filename=package://robot_control/robot_description/meshes/stl/encaix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 scale=1.0 1.0 1.0
- link link_acker_front_right: geometry visual mesh filename=package://robot_control/robot_description/meshes/stl/encaix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 scale=1.0 1.0 1.0
- link link_wheel_front_left: geometry collision cylinder length=0.05 radius=0.05; visual mesh filename=package://robot_control/robot_description/meshes/stl/wheel_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 scale=1.0 1.0 1.0
- link link_wheel_front_right: geometry collision cylinder length=0.05 radius=0.05; visual mesh filename=package://robot_control/robot_description/meshes/stl/wheel_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 scale=1.0 1.0 1.0
- link link_wheel_rear_left: geometry collision cylinder length=0.05 radius=0.05; visual mesh filename=package://robot_control/robot_description/meshes/stl/wheel_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 scale=1.0 1.0 1.0
- link link_wheel_rear_right: geometry collision cylinder length=0.05 radius=0.05; visual mesh filename=package://robot_control/robot_description/meshes/stl/wheel_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 scale=1.0 1.0 1.0

File: Jetson/catkin_ws/src/robot_control/robot_description/urdf/Ackermann_robot.urdf.xacro (robot description, xacro)
@@ -1,5 +1,5 @@
 <?xml version="1.0" encoding="utf-8"?>
 <robot name="Ackermann_robot" xmlns:xacro="http://ros.org/wiki/xacro">
-    <xacro:property name="package_name" value="ackermann_vehicle_description"/>
+    <xacro:property name="package_name" value="robot_control"/>
     <xacro:include filename="base.xacro"/>
     <xacro:include filename="wheels_links.xacro"/>
@@ -15,3 +15,29 @@
         </plugin>
     </gazebo>
+    <gazebo reference="imu_link">
+    <sensor type="imu" name="imu_sensor">
+        <pose>0 0 0 0 0 0</pose> <!-- pode ajustar caso queira deslocar -->
+        <always_on>true</always_on>
+        <update_rate>100.0</update_rate>
+        <imu>
+        <noise>
+            <type>gaussian</type>
+            <rate>
+            <mean>0.0</mean>
+            <stddev>0.0001</stddev>
+            </rate>
+            <accel>
+            <mean>0.0</mean>
+            <stddev>0.0001</stddev>
+            </accel>
+        </noise>
+        </imu>
+        <plugin name="imu_plugin" filename="libgazebo_ros_imu.so">
+        <robotNamespace>/</robotNamespace>
+        <bodyName>imu_link</bodyName>
+        <topicName>imu/data</topicName>
+        <frameName>imu_link</frameName>
+        </plugin>
+    </sensor>
+    </gazebo>
 </robot>

File: Jetson/catkin_ws/src/robot_control/robot_description/urdf/base.xacro (robot description, xacro)
@@ -5,5 +5,5 @@
     <!--</xacro:macro>-->
     <!--<xacro:chassi_link name="chassi_link"/>-->
-    <xacro:property name="BASE" value="package://${package_name}/robot/meshes/stl/Base.stl"/>
+    <xacro:property name="BASE" value="package://${package_name}/robot_description/meshes/stl/Base.stl"/>
     <material name="base_color">
       <color rgba="0.8 0.8 0.8 1.0"/>

File: Jetson/catkin_ws/src/robot_control/robot_description/urdf/torno_arckermann_links.xacro (robot description, xacro)
@@ -1,6 +1,6 @@
 <?xml version="1.0" encoding="utf-8"?>
 <robot xmlns:xacro="http://ros.org/wiki/xacro">
-    <xacro:property name="FL_TORNO" value="package://${package_name}/robot/meshes/stl/encaixe_front_left.stl"/>
-    <xacro:property name="FR_TORNO" value="package://${package_name}/robot/meshes/stl/encaixe_front_right.stl"/>
+    <xacro:property name="FL_TORNO" value="package://${package_name}/robot_description/meshes/stl/encaixe_front_left.stl"/>
+    <xacro:property name="FR_TORNO" value="package://${package_name}/robot_description/meshes/stl/encaixe_front_right.stl"/>
     <xacro:macro name="default_torno_inertials">
       <mass value="0.15"/>

File: Jetson/catkin_ws/src/robot_control/robot_description/urdf/wheels_links.xacro (robot description, xacro)
@@ -1,8 +1,8 @@
 <?xml version="1.0" encoding="utf-8"?>
 <robot xmlns:xacro="http://ros.org/wiki/xacro">
-    <xacro:property name="FL_WHEEL" value="package://${package_name}/robot/meshes/stl/wheel_front_left.stl"/>
-    <xacro:property name="FR_WHEEL" value="package://${package_name}/robot/meshes/stl/wheel_front_right.stl"/>
-    <xacro:property name="RL_WHEEL" value="package://${package_name}/robot/meshes/stl/wheel_rear_left.stl"/>
-    <xacro:property name="RR_WHEEL" value="package://${package_name}/robot/meshes/stl/wheel_rear_right.stl"/>
+    <xacro:property name="FL_WHEEL" value="package://${package_name}/robot_description/meshes/stl/wheel_front_left.stl"/>
+    <xacro:property name="FR_WHEEL" value="package://${package_name}/robot_description/meshes/stl/wheel_front_right.stl"/>
+    <xacro:property name="RL_WHEEL" value="package://${package_name}/robot_description/meshes/stl/wheel_rear_left.stl"/>
+    <xacro:property name="RR_WHEEL" value="package://${package_name}/robot_description/meshes/stl/wheel_rear_right.stl"/>
     <xacro:macro name="default_wheel_inertials">
       <mass value="0.15"/>
