Commit message: Adicionada IMU na simulação e criado o link e junta do Lidar

File: Jetson/catkin_ws/src/robot_control/robot_description/urdf/Ackermann_robot.urdf.xacro (robot description, xacro)
@@ -15,29 +15,3 @@
         </plugin>
     </gazebo>
-    <gazebo reference="imu_link">
-    <sensor type="imu" name="imu_sensor">
-        <pose>0 0 0 0 0 0</pose> <!-- pode ajustar caso queira deslocar -->
-        <always_on>true</always_on>
-        <update_rate>100.0</update_rate>
-        <imu>
-        <noise>
-            <type>gaussian</type>
-            <rate>
-            <mean>0.0</mean>
-            <stddev>0.0001</stddev>
-            </rate>
-            <accel>
-            <mean>0.0</mean>
-            <stddev>0.0001</stddev>
-            </accel>
-        </noise>
-        </imu>
-        <plugin name="imu_plugin" filename="libgazebo_ros_imu.so">
-        <robotNamespace>/</robotNamespace>
-        <bodyName>imu_link</bodyName>
-        <topicName>imu/data</topicName>
-        <frameName>imu_link</frameName>
-        </plugin>
-    </sensor>
-    </gazebo>
 </robot>

File: Jetson/catkin_ws/src/robot_control/robot_description/urdf_teste/imu.xacro (robot description, xacro)
@@ -25,5 +25,5 @@
     </link>
     <joint name="imu_joint" type="fixed">
-        <origin xyz="0 0 0.07077" rpy="0 0 0"/>
+        <origin xyz="0.15 0 0.07077" rpy="0 0 0"/>
         <parent link="base_link" />
         <child link="imu_link" />

File: Jetson/catkin_ws/src/robot_control/robot_description/urdf_teste/steer_bot.urdf.xacro (robot description, xacro)
@@ -17,5 +17,6 @@
   <!-- Include xacro for inertials, materials and wheels -->
   <xacro:include filename="$(find robot_control)/robot_description/urdf_teste/wheel.xacro"/>
-  <!--<xacro:include filename="$(find robot_control)/robot_description/urdf_teste/imu.xacro"/>-->
+  <xacro:include filename="$(find robot_control)/robot_description/urdf_teste/imu.xacro"/>
+  <xacro:include filename="$(find robot_control)/robot_description/urdf_teste/lidar.xacro"/>
   <xacro:property name="robot_namespace" value="/steer_bot"/>
   <!-- Gazebo plugins -->
@@ -29,5 +30,4 @@
     </plugin>
   </gazebo>
-  <!--
   <gazebo reference="imu_link">
     <sensor type="imu" name="imu_sensor">
@@ -35,4 +35,5 @@
       <always_on>true</always_on>
       <update_rate>100.0</update_rate>
+      <visualize>true</visualize>
       <imu>
         <noise>
@@ -48,5 +49,5 @@
         </noise>
       </imu>
-      <plugin name="imu_plugin" filename="libgazebo_ros_imu.so">
+      <plugin name="imu_plugin" filename="libgazebo_ros_imu_sensor.so">
         <robotNamespace>/</robotNamespace>
         <bodyName>imu_link</bodyName>
@@ -56,5 +57,4 @@
     </sensor>
   </gazebo>
-  -->
   <!-- Math constants -->
   <xacro:property name="deg_to_rad" value="0.01745329251994329577"/>
@@ -75,4 +75,7 @@
   <xacro:property name="axle_offset" value="0.05" />
   <xacro:property name="steer_offset" value="0.02" />
+  <!-- Lidar dimensions -->
+  <xacro:property name="lidar_radius" value="0.08" />
+  <xacro:property name="lidar_length" value="0.04" />
   <!-- Base link -->
   <link name="base_link">
@@ -163,4 +166,13 @@
     <origin xyz="${-base_length/2+axle_offset} ${+base_width/2+axle_offset} 0" rpy="${-90 * deg_to_rad} 0 0"/>
   </xacro:rear_wheel_lr>
+  <!-- RPLidar -->
+  <xacro:rplidar
+    name="rplidar"
+    parent="base_link"
+    base_length="${base_length}"
+    base_height="${base_height}"
+    radius="${lidar_radius}"
+    length="${lidar_length}">
+  </xacro:rplidar>
   <!-- Colour -->
   <gazebo reference="base_link">

Commit message: Mudanças do fernandão + hw_interface

File: Jetson/catkin_ws/src/robot_control/robot_description/urdf/Ackermann_robot.urdf.xacro (robot description, xacro)
@@ -9,4 +9,5 @@
     <xacro:include filename="imu.xacro"/>
     <xacro:include filename="transmissions.xacro"/>
+    <xacro:include filename="lidar.xacro"/>
     <gazebo>
         <plugin name="gazebo_ros_control" filename="libgazebo_ros_control.so">

File: Jetson/catkin_ws/src/robot_control/robot_description/urdf/lidar.xacro (robot description, xacro)
@@ -1,3 +1,28 @@
 <?xml version="1.0" encoding="utf-8"?>
 <robot xmlns:xacro="http://ros.org/wiki/xacro">
+    <!-- Parâmetros configuráveis do LiDAR -->
+    <xacro:property name="lidar_radius" value="0.038"/>   <!-- 5 cm de raio -->
+    <xacro:property name="lidar_height" value="0.041"/>   <!-- 2 cm de altura -->
+    <!-- Link do LiDAR -->
+    <link name="lidar_link">
+        <visual>
+            <geometry>
+                <cylinder radius="${lidar_radius}" length="${lidar_height}"/>
+            </geometry>
+            <material name="Grey">
+                <color rgba="0.6 0.6 0.6 1.0"/>
+            </material>
+        </visual>
+        <collision>
+            <geometry>
+                <cylinder radius="${lidar_radius}" length="${lidar_height}"/>
+            </geometry>
+        </collision>
+    </link>
+    <!-- Local para você criar a junta entre o LiDAR e o link pai -->
+    <joint name="lidar_joint" type="fixed">
+        <parent link="base_link"/>
+        <child link="lidar_link"/>
+        <origin xyz="0 0.02945 0" rpy="0 0 0"/>  <!-- Ajuste a posição e orientação do LiDAR -->
+    </joint>
 </robot>
