Commit message: Adicionado funcionamento do Lidar na simulação

File: Jetson/catkin_ws/src/robot_control/robot_description/urdf_teste/lidar.xacro (robot description, xacro)
@@ -33,6 +33,6 @@
     <joint name="${name}_joint" type="fixed">
       <parent link="${parent}"/>
-      <child link="rplidar_link"/>
-      <origin xyz="${base_length/2 + radius} 0 ${base_height/2 - length/2}" rpy="0 0 0"/>
+      <child link="${name}_link"/>
+      <origin xyz="${base_length/2 + radius} 0 ${base_height/2 + length/2}" rpy="0 0 0"/>
     </joint>
   </xacro:macro>

File: Jetson/catkin_ws/src/robot_control/robot_description/urdf_teste/steer_bot.urdf.xacro (robot description, xacro)
@@ -54,4 +54,35 @@
         <topicName>imu/data</topicName>
         <frameName>imu_link</frameName>
+      </plugin>
+    </sensor>
+  </gazebo>
+  <gazebo reference="rplidar_link">
+    <sensor name="rplidar" type="ray">
+      <pose>0 0 0 0 0 0</pose>
+      <visualize>true</visualize>
+      <update_rate>40</update_rate>
+      <ray>
+        <scan>
+          <horizontal>
+            <samples>720</samples>
+            <resolution>1</resolution>
+            <min_angle>-1.570796</min_angle>
+            <max_angle>1.570796</max_angle>
+          </horizontal>
+        </scan>
+        <range>
+          <min>0.12</min>
+          <max>30.0</max>
+          <resolution>0.01</resolution>
+        </range>
+        <noise>
+          <type>gaussian</type>
+          <mean>0.0</mean>
+          <stddev>0.01</stddev>
+        </noise>
+      </ray>
+      <plugin name="gazebo_ros_laser" filename="libgazebo_ros_laser.so">
+        <topicName>scan</topicName>
+        <frameName>rplidar_link</frameName>
       </plugin>
     </sensor>
